File: DataManager_Shield/aux_pins.kicad_sch (KiCad schematic)
At the start: 1 part, among them J2 aux_pin

Commit message: Routing PCB Finished
Connections:
- net ADC1_IN2 is gone; now on net MCOR_Speed_Control_IN_to_MCU: J2.36 (Pin_36)
- net MCOR_Speed_Control_IN_to_MCU: no longer J2.35 (Pin_35)
- new net ADC1_IN3: J2.35 (Pin_35)
Changed lines of the file:
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@@
+	)
+	(no_connect
+		(at 123.19 118.11)
 	)
 	(no_connect
@@
 	(no_connect
 		(at 166.37 102.87)
-	)
-	(no_connect
-		(at 165.1 118.11)
 	)
 	(no_connect
@@
 	(hierarchical_label "MCOR_Speed_Control_IN_to_MCU"
 		(shape input)
-		(at 123.19 118.11 180)
-		(effects
-			(font
-				(size 1.27 1.27)
-			)
-			(justify right)
-		)
-	)
+		(at 165.1 118.11 0)
+		(effects
+			(font
+				(size 1.27 1.27)
+			)
+			(justify left)
+		)
+	)
