File: DataManager_Shield/aux_pins.kicad_sch (KiCad schematic)
At the start: 1 part, among them J2 aux_pin

Commit message: Data logger board Major Fixes - Remove Speed Sensor's LED and increase R value - Remove Pedal level reader - Remove aux pin header from BoM, self soldering
Parts:
- J2: now not fitted; now left out of the parts list
Connections:
- net MCOR_Speed_Control_IN_to_MCU renamed ADC1_IN2
- no-connect marks 22 -> 23
Changed lines of the file:
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@@
+	)
+	(no_connect
+		(at 165.1 118.11)
 	)
 	(no_connect
@@
 			)
 			(justify right)
-		)
-	)
-	(hierarchical_label "MCOR_Speed_Control_IN_to_MCU"
-		(shape input)
-		(at 165.1 118.11 0)
-		(effects
-			(font
-				(size 1.27 1.27)
-			)
-			(justify left)
 		)
 	)
@@
 		(body_style 1)
 		(exclude_from_sim no)
-		(in_bom yes)
+		(in_bom no)
 		(on_board yes)
 		(in_pos_files yes)
-		(dnp no)
+		(dnp yes)
 		(fields_autoplaced yes)
 		(property "Reference" "J2"
