File: DataManager_Shield/DataManager_Shield.kicad_pcb (KiCad board)
At the start: 4 copper layers, 78 x 70 mm, 63 parts, among them J1 CAR_IN, J2 aux_pin, J3 CAR_OUT, J4 Mode_Selector, K1 IM03, K2 IM03, Q10 AO3400A, Q9 AO3400A, U1 TLP291-4, U2 MCP4725xxx-xCH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

Commit message: Routing PCB Finished
Parts:
- added R30: 4.7k, Resistor_SMD:R_0603_1608Metric, F.Cu at (133.0, 96.2)
- added R31: 4.7k, Resistor_SMD:R_0603_1608Metric, F.Cu at (133.0, 97.8)
- added TP9: MCOR_Speed_Control_IN, TestPoint:TestPoint_Pad_1.0x1.0mm, F.Cu at (98.5, 72.0)
- added U4: PCA9306, Package_SO:VSSOP-8_2.3x2mm_P0.5mm, F.Cu at (130.2, 95.4)
- added kibuzzard-6A36AE6B: G***, kibuzzard-6A36AE6B, F.Cu at (90.5, 52.0)
- added kibuzzard-6A36AE7E: G***, kibuzzard-6A36AE7E, F.Cu at (144.0, 52.0)
- added kibuzzard-6A36AEB2: G***, kibuzzard-6A36AEB2, F.Cu at (103.8, 56.6)
- added kibuzzard-6A36B03F: G***, kibuzzard-6A36B03F, F.Cu at (121.5, 59.8)
- added kibuzzard-6A36B04E: G***, kibuzzard-6A36B04E, F.Cu at (122.0, 69.2)
- added kibuzzard-6A36B06A: G***, kibuzzard-6A36B06A, F.Cu at (122.4, 73.8)
- added kibuzzard-6A36B07D: G***, kibuzzard-6A36B07D, F.Cu at (107.5, 82.0)
- added kibuzzard-6A36B090: G***, kibuzzard-6A36B090, F.Cu at (98.5, 84.0)
- added kibuzzard-6A36B0C2: G***, kibuzzard-6A36B0C2, F.Cu at (97.5, 94.5)
- added kibuzzard-6A36B0D5: G***, kibuzzard-6A36B0D5, F.Cu at (133.0, 75.5)
- added kibuzzard-6A36B2C1: G***, kibuzzard-6A36B2C1, F.Cu at (102.5, 72.0)
- added kibuzzard-6A36C52F: G***, kibuzzard-6A36C52F, F.Cu at (116.8, 43.2)
- C1: value 100nF 50V -> 100nF 16V
- R26: value 20k -> 15k
- moved R17 101.8 mm to (104.0, 62.2), turned to 180 degrees
- moved R10 95.7 mm to (123.6, 62.8), turned to 180 degrees
- moved R9 92.9 mm to (126.6, 62.8), turned to 180 degrees
- moved R18 91.5 mm to (104.0, 65.4), turned to 180 degrees
- moved R21 90.8 mm to (104.0, 68.6), turned to 180 degrees
- moved R20 87.1 mm to (117.0, 67.0)
- moved R22 85.8 mm to (117.0, 71.6)
- moved R26 81.9 mm to (140.2, 96.6)
- moved R15 76.1 mm to (94.0, 93.8), turned to 180 degrees
- moved R19 74.1 mm to (117.0, 63.0)
- moved D1 73.9 mm to (133.4, 59.6)
- moved R14 73.0 mm to (132.5, 91.8), turned to 90 degrees
- moved R16 72.3 mm to (119.8, 87.6)
- moved R29 71.8 mm to (103.0, 86.4)
- moved R13 71.2 mm to (134.0, 92.8), turned to 90 degrees
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Connections:
- D3 pad 3: /aux_pins/ADC1_IN3 -> /aux_pins/ADC1_IN2
- R13 pad 1: /aux_pins/PA9 -> Net-(U2-SCL)
- R14 pad 1: /aux_pins/PA8 -> Net-(U2-SDA)
- R26 pad 1: /aux_pins/ADC1_IN3 -> /aux_pins/ADC1_IN2
- R5 pad 2: /aux_pins/ADC1_IN3 -> /aux_pins/ADC1_IN2
- U2 pad 4: /aux_pins/PA8 -> Net-(U2-SDA)
- U2 pad 5: /aux_pins/PA9 -> Net-(U2-SCL)
Routing:
- net /Relays/MCOR_Speed_Control_IN: track 0.00 -> 155.9 mm, vias 0 -> 6
- net /aux_pins/PA10: track 0.00 -> 145.5 mm, vias 0 -> 2
- net +5V: track 0.00 -> 118.0 mm, vias 0 -> 6
- net /Relays/Backward_IN: track 0.00 -> 117.2 mm, vias 0 -> 2
- net /Relays/Forward_IN: track 0.00 -> 101.5 mm, vias 0 -> 2
- net /Relays/Pedal_IN: track 0.00 -> 93.6 mm, vias 0 -> 2
- net /Relays/Power_Down/Charger_Interlock: track 0.00 -> 90.9 mm, vias 0 -> 1
- net +3V3: track 0.00 -> 85.8 mm, vias 0 -> 7
- net /aux_pins/PC6: track 0.00 -> 56.9 mm, vias 0 -> 2
- net /aux_pins/PC7: track 0.00 -> 55.1 mm, vias 0 -> 2
- net /aux_pins/PC8: track 0.00 -> 54.0 mm, vias 0 -> 2
- net GND: track 0.00 -> 46.1 mm, vias 0 -> 21
- net /Relays/MCOR_Speed_Control_from_MCU: track 0.00 -> 45.3 mm
- net /Relays/Forward_OUT_from_MCU: track 0.00 -> 40.5 mm
- net /Relays/Pedal_OUT: track 0.00 -> 33.1 mm
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- added copper zone on B.Cu, net GND
- added copper zone on F.Cu, net GND
- added copper zone on In1.Cu, net GND
- added copper zone on In2.Cu, net GND

Commit message: fix silk screen and fix offset rotation for fabrication
Parts:
- removed kibuzzard-6A36AEB2: G***, kibuzzard-6A36AEB2
- added kibuzzard-6A36CCD0: G***, kibuzzard-6A36CCD0, F.Cu at (104.8, 56.6)

Commit message: up
Routing:
- net /Relays/MCOR_Speed_Control_IN: track 155.9 -> 154.5 mm
- net /Relays/Speed_Sensor: track 79.4 -> 78.2 mm
- net /Relays/Key_Switch_In: track 118.7 -> 117.7 mm
- net /Relays/ Speed_Sensor_Supply_Out / about_15V: track 97.1 -> 96.3 mm
- net /Relays/Power_Down/Charger_Interlock: track 90.9 -> 90.3 mm
