File: DataManager_Shield/DataManager_Shield.kicad_pcb (KiCad board)
At the start: 4 copper layers, 78 x 70 mm, 74 parts, among them J1 CAR_IN, J2 aux_pin, J3 CAR_OUT, J4 Mode_Selector, K1 IM03, K2 IM03, Q10 AO3400A, Q9 AO3400A, U1 TLP291-4, U2 MCP4725xxx-xCH, U3 TLP291-4, U4 PCA9306

Commit message: Isolate GND for Datamanager Shield
Parts:
- removed U4: PCA9306, Package_SO:VSSOP-8_2.3x2mm_P0.5mm
- added C2: 100nF 16V, Capacitor_SMD:C_0402_1005Metric, F.Cu at (127.5, 92.5)
- added U5: ADuM1250, Package_SO:SOIC-8_3.9x4.9mm_P1.27mm, F.Cu at (132.1, 94.0)
- moved R30 6.96 mm to (126.2, 94.7), turned to 90 degrees
- moved R13 5.63 mm to (139.0, 95.4), turned to -90 degrees
- moved R14 5.51 mm to (137.3, 94.5), turned to -90 degrees
- moved U2 5.28 mm to (142.0, 94.5)
- moved C1 4.42 mm to (142.0, 96.7), turned to 180 degrees
- moved R31 1.80 mm to (131.2, 97.8)
Connections:
- C1 pad 1: +5V -> /Relays/Pot_High_Out/5V_throttle_ref
- C1 pad 2: GND -> B-
- R13 pad 2: +5V -> /Relays/Pot_High_Out/5V_throttle_ref
- R14 pad 2: +5V -> /Relays/Pot_High_Out/5V_throttle_ref
- R30 pad 1: /aux_pins/PA9 -> /aux_pins/PA8
- R31 pad 1: /aux_pins/PA8 -> /aux_pins/PA9
- U2 pad 2: GND -> B-
- U2 pad 3: +5V -> /Relays/Pot_High_Out/5V_throttle_ref
- U2 pad 6: GND -> B-
Routing:
- net +5V: track 118.0 -> 94.3 mm, vias 6 -> 3
- net B-: track 145.7 -> 168.8 mm, vias 8 -> 10
- net /Relays/Pot_High_Out/5V_throttle_ref: track 102.6 -> 123.5 mm, vias 0 -> 3
- net /aux_pins/PA8: track 7.52 -> 15.2 mm
- net /Relays/MCOR_Speed_Control_from_MCU: track 45.3 -> 40.5 mm
- net GND: track 29.0 -> 25.5 mm, vias 12 -> 11
- net +3V3: track 72.4 -> 75.0 mm, vias 6 -> 5
- net /aux_pins/PA9: track 6.95 -> 9.24 mm
- net Net-(U2-SCL): track 7.68 -> 6.34 mm
- net /aux_pins/PA15: track 23.1 -> 24.1 mm
- net Net-(U2-SDA): track 5.74 -> 6.47 mm
