File: DataManager_Shield/Relays.kicad_sch (KiCad schematic)
At the start: 58 parts, among them J1 CAR_IN, J3 CAR_OUT, J4 Mode_Selector, K1 IM03, K2 IM03, Q10 AO3400A, Q9 AO3400A, U1 TLP291-4, U2 MCP4725xxx-xCH, U3 TLP291-4

Commit message: Routing PCB Finished
Parts:
- added R30, R31: 4.7k, Resistor_SMD:R_0603_1608Metric, symbol Device:R_Small
- added TP9: MCOR_Speed_Control_IN, TestPoint:TestPoint_Pad_1.0x1.0mm, symbol Connector:TestPoint
- added U4: PCA9306, Package_SO:VSSOP-8_2.3x2mm_P0.5mm, symbol Interface:PCA9306
- C1: value 100nF 50V -> 100nF 16V
- J1, J3: FT Rotation Offset (none) -> 180
- J4: FT Rotation Offset (none) -> 180; JLCPCB Part # C157931 -> C163035
- K1, K2: FT Rotation Offset (none) -> 270
- R26: value 20k -> 15k; JLCPCB Part # C4184 -> C22809
- U2: FT Rotation Offset (none) -> 90
Connections:
- net +3V3: now also R30.2, R31.2, U4.2 (VREF1), U4.8 (EN)
- net +5V: now also U4.7 (VREF2)
- net GND: now also U4.1 (GND)
- net MCOR_Speed_Control_IN: now also TP9.1
- net MCP4725_SCL: now also R30.1, U4.3 (SCL1); no longer R13.1, U2.5 (SCL)
- net MCP4725_SDA: now also R31.1, U4.4 (SDA1); no longer R14.1, U2.4 (SDA)
- new net: R14.1, U2.4 (SDA), U4.5 (SDA2)
- new net: R13.1, U2.5 (SCL), U4.6 (SCL2)
Other:
- moved on the sheet: C1, R13, R14, TP7, U2

Commit message: up
Parts:
- R12, R15, R16, R5, R6, R7, R8, R9: JLCPCB Part # C25804 -> C130232
Changed lines of the file:
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@@
 			)
 		)
-		(property "JLCPCB Part #" "C25804"
+		(property "JLCPCB Part #" "C130232"
 			(at 111.76 219.71 0)
 			(hide yes)
@@
 			)
 		)
-		(property "JLCPCB Part #" "C25804"
+		(property "JLCPCB Part #" "C130232"
 			(at 181.61 200.66 0)
 			(hide yes)
@@
 			)
 		)
-		(property "JLCPCB Part #" "C25804"
+		(property "JLCPCB Part #" "C130232"
 			(at 180.34 168.91 0)
 			(hide yes)
@@
 			)
 		)
-		(property "JLCPCB Part #" "C25804"
+		(property "JLCPCB Part #" "C130232"
 			(at 180.34 113.03 0)
 			(hide yes)
@@
 			)
 		)
-		(property "JLCPCB Part #" "C25804"
+		(property "JLCPCB Part #" "C130232"
 			(at 173.99 76.2 0)
 			(hide yes)
@@
 			)
 		)
-		(property "JLCPCB Part #" "C25804"
+		(property "JLCPCB Part #" "C130232"
 			(at 76.2 182.88 0)
 			(hide yes)
@@
 			)
 		)
-		(property "JLCPCB Part #" "C25804"
+		(property "JLCPCB Part #" "C130232"
 			(at 180.34 140.97 0)
 			(hide yes)
@@
 			)
 		)
-		(property "JLCPCB Part #" "C25804"
+		(property "JLCPCB Part #" "C130232"
 			(at 76.2 129.54 0)
 			(hide yes)
