File: DataManager_Shield/Relays.kicad_sch (KiCad schematic)
At the start: 62 parts, among them J1 CAR_IN, J3 CAR_OUT, J4 Mode_Selector, K1 IM03, K2 IM03, Q10 AO3400A, Q9 AO3400A, U1 TLP291-4, U2 MCP4725xxx-xCH, U3 TLP291-4, U4 PCA9306

Commit message: Fix PCB Isolate GND
Parts:
- added J6: Screw_Terminal_01x02, TerminalBlock_MetzConnect:TerminalBlock_MetzConnect_Type011_RT05502HBLC_1x02_P5.00mm_Horizontal, symbol Connector:Screw_Terminal_01x02
- R26: value 15k -> 1.5M
- R5: value 10k -> 1M
Connections:
- net Pot_Low_out is gone; now on net GND: J1.3 (Pin_3), J3.3 (Pin_3)
- net GND: no longer R19.2, R20.2, R22.2
- new net B-: J6.1 (Pin_1), J6.2 (Pin_2), R19.2, R20.2, R22.2

Commit message: Update
Parts:
- J6: value Screw_Terminal_01x02 -> B-
Connections:
- net B-: now also U1.4, U1.6, U1.8
- net GND: no longer U1.4, U1.6, U1.8
Changed lines of the file:
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@@
 	(symbol
 		(lib_id "power:GND")
+		(at 161.29 110.49 0)
+		(unit 1)
+		(body_style 1)
+		(exclude_from_sim no)
+		(in_bom yes)
+		(on_board yes)
+		(in_pos_files yes)
+		(dnp no)
+		(property "Reference" "#PWR054"
+			(at 161.29 116.84 0)
+			(hide yes)
+			(show_name no)
+			(do_not_autoplace no)
+			(effects
+				(font
+					(size 1.27 1.27)
+				)
+			)
+		)
+		(property "Value" "B-"
+			(at 161.29 114.3 0)
+			(show_name no)
+			(do_not_autoplace no)
+			(effects
+				(font
+					(size 1.27 1.27)
+				)
+			)
+		)
+		(property "Footprint" ""
+			(at 161.29 110.49 0)
+			(hide yes)
+			(show_name no)
+			(do_not_autoplace no)
+			(effects
+				(font
+					(size 1.27 1.27)
+				)
+			)
+		)
+		(property "Datasheet" ""
+			(at 161.29 110.49 0)
+			(hide yes)
+			(show_name no)
+			(do_not_autoplace no)
+			(effects
+				(font
+					(size 1.27 1.27)
+				)
+			)
+		)
+		(property "Description" "Power symbol creates a global label with name \"GND\" , ground"
+			(at 161.29 110.49 0)
+			(hide yes)
+			(show_name no)
+			(do_not_autoplace no)
+			(effects
+				(font
+					(size 1.27 1.27)
+				)
+			)
+		)
+		(pin "1"
+		)
+		(instances
+			(project "DataManager_Shield"
+				(path "/74a95295-856f-462a-99dc-2eba26429db4/3f3103c2-6ce4-4371-b040-f30e7a818592"
+					(reference "#PWR054")
+					(unit 1)
+				)
+			)
+		)
+	)
+	(symbol
+		(lib_id "power:GND")
 		(at 92.71 38.1 0)
 		(unit 1)
@@
 	(symbol
 		(lib_id "power:GND")
+		(at 161.29 166.37 0)
+		(unit 1)
+		(body_style 1)
+		(exclude_from_sim no)
+		(in_bom yes)
+		(on_board yes)
+		(in_pos_files yes)
+		(dnp no)
+		(property "Reference" "#PWR056"
+			(at 161.29 172.72 0)
+			(hide yes)
+			(show_name no)
+			(do_not_autoplace no)
+			(effects
+				(font
+					(size 1.27 1.27)
+				)
+			)
+		)
+		(property "Value" "B-"
+			(at 161.29 170.18 0)
+			(show_name no)
+			(do_not_autoplace no)
+			(effects
+				(font
+					(size 1.27 1.27)
+				)
+			)
+		)
+		(property "Footprint" ""
+			(at 161.29 166.37 0)
+			(hide yes)
+			(show_name no)
+			(do_not_autoplace no)
+			(effects
+				(font
+					(size 1.27 1.27)
+				)
+			)
+		)
+		(property "Datasheet" ""
+			(at 161.29 166.37 0)
+			(hide yes)
+			(show_name no)
+			(do_not_autoplace no)
+			(effects
+				(font
+					(size 1.27 1.27)
+				)
+			)
+		)
+		(property "Description" "Power symbol creates a global label with name \"GND\" , ground"
+			(at 161.29 166.37 0)
+			(hide yes)
+			(show_name no)
+			(do_not_autoplace no)
+			(effects
+				(font
+					(size 1.27 1.27)
+				)
+			)
+		)
+		(pin "1"
+		)
+		(instances
+			(project "DataManager_Shield"
+				(path "/74a95295-856f-462a-99dc-2eba26429db4/3f3103c2-6ce4-4371-b040-f30e7a818592"
+					(reference "#PWR056")
+					(unit 1)
+				)
+			)
+		)
+	)
+	(symbol
+		(lib_id "power:GND")
 		(at 271.78 147.32 0)
 		(unit 1)
@@
 			)
 		)
-		(property "Value" "Screw_Terminal_01x02"
+		(property "Value" "B-"
 			(at 281.94 246.3799 0)
 			(show_name no)
@@
 	(symbol
 		(lib_id "power:GND")
-		(at 161.29 166.37 0)
-		(unit 1)
-		(body_style 1)
-		(exclude_from_sim no)
-		(in_bom yes)
-		(on_board yes)
-		(in_pos_files yes)
-		(dnp no)
-		(fields_autoplaced yes)
-		(property "Reference" "#PWR011"
-			(at 161.29 172.72 0)
-			(hide yes)
-			(show_name no)
-			(do_not_autoplace no)
-			(effects
-				(font
-					(size 1.27 1.27)
-				)
-			)
-		)
-		(property "Value" "GND"
-			(at 161.29 171.45 0)
-			(show_name no)
-			(do_not_autoplace no)
-			(effects
-				(font
-					(size 1.27 1.27)
-				)
-			)
-		)
-		(property "Footprint" ""
-			(at 161.29 166.37 0)
-			(hide yes)
-			(show_name no)
-			(do_not_autoplace no)
-			(effects
-				(font
-					(size 1.27 1.27)
-				)
-			)
-		)
-		(property "Datasheet" ""
-			(at 161.29 166.37 0)
-			(hide yes)
-			(show_name no)
-			(do_not_autoplace no)
-			(effects
-				(font
-					(size 1.27 1.27)
-				)
-			)
-		)
-		(property "Description" "Power symbol creates a global label with name \"GND\" , ground"
-			(at 161.29 166.37 0)
-			(hide yes)
-			(show_name no)
-			(do_not_autoplace no)
-			(effects
-				(font
-					(size 1.27 1.27)
-				)
-			)
-		)
-		(pin "1"
-		)
-		(instances
-			(project "DataManager_Shield"
-				(path "/74a95295-856f-462a-99dc-2eba26429db4/3f3103c2-6ce4-4371-b040-f30e7a818592"
-					(reference "#PWR011")
-					(unit 1)
-				)
-			)
-		)
-	)
-	(symbol
-		(lib_id "power:GND")
-		(at 161.29 138.43 0)
-		(unit 1)
-		(body_style 1)
-		(exclude_from_sim no)
-		(in_bom yes)
-		(on_board yes)
-		(in_pos_files yes)
-		(dnp no)
-		(fields_autoplaced yes)
-		(property "Reference" "#PWR09"
-			(at 161.29 144.78 0)
-			(hide yes)
-			(show_name no)
-			(do_not_autoplace no)
-			(effects
-				(font
-					(size 1.27 1.27)
-				)
-			)
-		)
-		(property "Value" "GND"
-			(at 161.29 143.51 0)
-			(show_name no)
-			(do_not_autoplace no)
-			(effects
-				(font
-					(size 1.27 1.27)
-				)
-			)
-		)
-		(property "Footprint" ""
-			(at 161.29 138.43 0)
-			(hide yes)
-			(show_name no)
-			(do_not_autoplace no)
-			(effects
-				(font
-					(size 1.27 1.27)
-				)
-			)
-		)
-		(property "Datasheet" ""
-			(at 161.29 138.43 0)
-			(hide yes)
-			(show_name no)
-			(do_not_autoplace no)
-			(effects
-				(font
-					(size 1.27 1.27)
-				)
-			)
-		)
-		(property "Description" "Power symbol creates a global label with name \"GND\" , ground"
-			(at 161.29 138.43 0)
-			(hide yes)
-			(show_name no)
-			(do_not_autoplace no)
-			(effects
-				(font
-					(size 1.27 1.27)
-				)
-			)
-		)
-		(pin "1"
-		)
-		(instances
-			(project "DataManager_Shield"
-				(path "/74a95295-856f-462a-99dc-2eba26429db4/3f3103c2-6ce4-4371-b040-f30e7a818592"
-					(reference "#PWR09")
-					(unit 1)
-				)
-			)
-		)
-	)
-	(symbol
-		(lib_id "power:GND")
 		(at 87.63 186.69 0)
 		(unit 1)
@@
 	)
 	(symbol
-		(lib_id "Diode:SS12")
-		(at 102.87 173.99 180)
+		(lib_id "power:GND")
+		(at 161.29 138.43 0)
 		(unit 1)
 		(body_style 1)
@@
 		(in_pos_files yes)
 		(dnp no)
-		(property "Reference" "D2"
-			(at 103.124 169.164 0)
-			(show_name no)
-			(do_not_autoplace no)
-			(effects
-				(font
-					(size 1.27 1.27)
-				)
-			)
-		)
-		(property "Value" "SS12"
-			(at 103.124 171.196 0)
+		(property "Reference" "#PWR055"
+			(at 161.29 144.78 0)
+			(hide yes)
 			(show_name no)
 			(do_not_autoplace no)
@@
 			)
 		)
-		(property "Footprint" "Diode_SMD:D_SMA"
-			(at 102.87 169.545 0)
-			(hide yes)
+		(property "Value" "B-"
+			(at 161.29 142.24 0)
 			(show_name no)
 			(do_not_autoplace no)
@@
 			)
 		)
-		(property "Datasheet" "https://www.vishay.com/docs/88746/ss12.pdf"
-			(at 102.87 173.99 0)
+		(property "Footprint" ""
+			(at 161.29 138.43 0)
 			(hide yes)
 			(show_name no)
@@
 			)
 		)
-		(property "Description" "20V 1A Schottky Diode, SMA"
-			(at 102.87 173.99 0)
+		(property "Datasheet" ""
+			(at 161.29 138.43 0)
 			(hide yes)
 			(show_name no)
@@
 			)
 		)
-		(property "JLCPCB Part #" "C18199177"
-			(at 102.87 173.99 0)
+		(property "Description" "Power symbol creates a global label with name \"GND\" , ground"
+			(at 161.29 138.43 0)
 			(hide yes)
 			(show_name no)
@@
 		(pin "1"
 		)
-		(pin "2"
-		)
 		(instances
 			(project "DataManager_Shield"
 				(path "/74a95295-856f-462a-99dc-2eba26429db4/3f3103c2-6ce4-4371-b040-f30e7a818592"
-					(reference "D2")
+					(reference "#PWR055")
 					(unit 1)
 				)
@@
 	)
 	(symbol
-		(lib_id "power:GND")
-		(at 161.29 110.49 0)
+		(lib_id "Diode:SS12")
+		(at 102.87 173.99 180)
 		(unit 1)
 		(body_style 1)
@@
 		(in_pos_files yes)
 		(dnp no)
-		(property "Reference" "#PWR06"
-			(at 161.29 116.84 0)
-			(hide yes)
+		(property "Reference" "D2"
+			(at 103.124 169.164 0)
 			(show_name no)
 			(do_not_autoplace no)
@@
 			)
 		)
-		(property "Value" "GND"
-			(at 161.29 114.554 0)
+		(property "Value" "SS12"
+			(at 103.124 171.196 0)
 			(show_name no)
 			(do_not_autoplace no)
@@
 			)
 		)
-		(property "Footprint" ""
-			(at 161.29 110.49 0)
+		(property "Footprint" "Diode_SMD:D_SMA"
+			(at 102.87 169.545 0)
 			(hide yes)
 			(show_name no)
@@
 			)
 		)
-		(property "Datasheet" ""
-			(at 161.29 110.49 0)
+		(property "Datasheet" "https://www.vishay.com/docs/88746/ss12.pdf"
+			(at 102.87 173.99 0)
 			(hide yes)
 			(show_name no)
@@
 			)
 		)
-		(property "Description" "Power symbol creates a global label with name \"GND\" , ground"
-			(at 161.29 110.49 0)
+		(property "Description" "20V 1A Schottky Diode, SMA"
+			(at 102.87 173.99 0)
+			(hide yes)
+			(show_name no)
+			(do_not_autoplace no)
+			(effects
+				(font
+					(size 1.27 1.27)
+				)
+			)
+		)
+		(property "JLCPCB Part #" "C18199177"
+			(at 102.87 173.99 0)
 			(hide yes)
 			(show_name no)
@@
 		(pin "1"
 		)
+		(pin "2"
+		)
 		(instances
 			(project "DataManager_Shield"
 				(path "/74a95295-856f-462a-99dc-2eba26429db4/3f3103c2-6ce4-4371-b040-f30e7a818592"
-					(reference "#PWR06")
+					(reference "D2")
 					(unit 1)
 				)

Commit message: Seperate out GND_SPEED
Connections:
- net GND: no longer D10.1 (K), U1.2
- net Speed_Sensor_Return renamed GND_SPEED
- net GND_SPEED: now also D10.1 (K), U1.2
Other:
- moved on the sheet: J3
Changed lines of the file:
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@@
 	(text "Reclamp connector"
 		(exclude_from_sim no)
-		(at 240.792 51.308 0)
+		(at 281.432 52.578 0)
 		(effects
 			(font
@@
 	)
 	(no_connect
-		(at 233.68 38.1)
+		(at 274.32 39.37)
 	)
 	(no_connect
@@
 	)
 	(no_connect
-		(at 246.38 35.56)
+		(at 287.02 36.83)
 	)
 	(wire
@@
 	(wire
 		(pts
-			(xy 196.85 40.64) (xy 233.68 40.64)
+			(xy 237.49 41.91) (xy 274.32 41.91)
 		)
 		(stroke
@@
 	(wire
 		(pts
-			(xy 246.38 43.18) (xy 287.02 43.18)
+			(xy 287.02 44.45) (xy 327.66 44.45)
 		)
 		(stroke
@@
 	(wire
 		(pts
-			(xy 196.85 30.48) (xy 233.68 30.48)
+			(xy 237.49 31.75) (xy 274.32 31.75)
 		)
 		(stroke
@@
 	(wire
 		(pts
-			(xy 246.38 30.48) (xy 251.46 30.48)
+			(xy 287.02 31.75) (xy 292.1 31.75)
 		)
 		(stroke
@@
 	(wire
 		(pts
-			(xy 196.85 48.26) (xy 233.68 48.26)
+			(xy 237.49 49.53) (xy 274.32 49.53)
 		)
 		(stroke
@@
 	(wire
 		(pts
-			(xy 196.85 45.72) (xy 233.68 45.72)
+			(xy 237.49 46.99) (xy 274.32 46.99)
 		)
 		(stroke
@@
 	(wire
 		(pts
-			(xy 287.02 33.02) (xy 246.38 33.02)
+			(xy 327.66 34.29) (xy 287.02 34.29)
 		)
 		(stroke
@@
 	(wire
 		(pts
-			(xy 246.38 40.64) (xy 287.02 40.64)
+			(xy 287.02 41.91) (xy 327.66 41.91)
 		)
 		(stroke
@@
 	(wire
 		(pts
-			(xy 246.38 38.1) (xy 287.02 38.1)
+			(xy 203.2 41.91) (xy 203.2 40.64)
+		)
+		(stroke
+			(width 0)
+			(type default)
+		)
+	)
+	(wire
+		(pts
+			(xy 287.02 39.37) (xy 327.66 39.37)
 		)
 		(stroke
@@
 	(wire
 		(pts
-			(xy 196.85 35.56) (xy 233.68 35.56)
+			(xy 237.49 36.83) (xy 274.32 36.83)
 		)
 		(stroke
@@
 	(wire
 		(pts
-			(xy 246.38 45.72) (xy 287.02 45.72)
+			(xy 287.02 46.99) (xy 327.66 46.99)
 		)
 		(stroke
@@
 	(wire
 		(pts
-			(xy 196.85 43.18) (xy 233.68 43.18)
+			(xy 237.49 44.45) (xy 274.32 44.45)
 		)
 		(stroke
@@
 	(wire
 		(pts
-			(xy 246.38 48.26) (xy 287.02 48.26)
+			(xy 287.02 49.53) (xy 327.66 49.53)
 		)
 		(stroke
@@
 	(wire
 		(pts
-			(xy 149.86 40.64) (xy 190.5 40.64)
+			(xy 149.86 40.64) (xy 203.2 40.64)
 		)
 		(stroke
@@
 	(wire
 		(pts
-			(xy 196.85 33.02) (xy 233.68 33.02)
+			(xy 237.49 34.29) (xy 274.32 34.29)
 		)
 		(stroke
@@
 	)
 	(label "Speed_Sensor"
-		(at 287.02 43.18 180)
+		(at 327.66 44.45 180)
 		(effects
 			(font
@@
 	)
 	(label " Speed_Sensor_Supply_Out / about_15V"
-		(at 287.02 45.72 180)
+		(at 327.66 46.99 180)
 		(effects
 			(font
@@
 	)
 	(label "Forward_OUT"
-		(at 196.85 48.26 0)
+		(at 237.49 49.53 0)
 		(effects
 			(font
@@
 	)
 	(label "Pot_Low_out"
-		(at 196.85 35.56 0)
+		(at 237.49 36.83 0)
 		(effects
 			(font
@@
 	)
 	(label "Speed_Sensor_Return"
-		(at 287.02 40.64 180)
+		(at 327.66 41.91 180)
 		(effects
 			(font
@@
 	)
 	(label "Pedal_OUT"
-		(at 196.85 43.18 0)
+		(at 237.49 44.45 0)
 		(effects
 			(font
@@
 	)
 	(label "Backward_OUT"
-		(at 287.02 48.26 180)
+		(at 327.66 49.53 180)
 		(effects
 			(font
@@
 	)
 	(label "Key_Switch_In"
-		(at 287.02 33.02 180)
+		(at 327.66 34.29 180)
 		(effects
 			(font
@@
 	)
 	(label "Power_Down/Charger_Interlock"
-		(at 196.85 40.64 0)
+		(at 237.49 41.91 0)
 		(effects
 			(font
@@
 	)
 	(label "Back_up_Alarm_Out"
-		(at 196.85 45.72 0)
+		(at 237.49 46.99 0)
 		(effects
 			(font
@@
 	)
 	(label "Main_Solenoid_Out"
-		(at 287.02 38.1 180)
+		(at 327.66 39.37 180)
 		(effects
 			(font
@@
 	)
 	(label "Pot_High_Out{slash}5V_throttle_ref"
-		(at 196.85 30.48 0)
+		(at 237.49 31.75 0)
 		(effects
 			(font
@@
 	)
 	(label "MCOR_Speed_Control_OUT"
-		(at 196.85 33.02 0)
+		(at 237.49 34.29 0)
 		(effects
 			(font
@@
 	(symbol
 		(lib_id "power:+48V")
-		(at 251.46 30.48 0)
+		(at 292.1 31.75 0)
 		(unit 1)
 		(body_style 1)
@@
 		(fields_autoplaced yes)
 		(property "Reference" "#PWR02"
-			(at 251.46 34.29 0)
+			(at 292.1 35.56 0)
 			(hide yes)
 			(show_name no)
@@
 		)
 		(property "Value" "+48V"
-			(at 251.46 25.4 0)
+			(at 292.1 26.67 0)
 			(show_name no)
 			(do_not_autoplace no)
@@
 		)
 		(property "Footprint" ""
-			(at 251.46 30.48 0)
+			(at 292.1 31.75 0)
 			(hide yes)
 			(show_name no)
@@
 		)
 		(property "Datasheet" ""
-			(at 251.46 30.48 0)
+			(at 292.1 31.75 0)
 			(hide yes)
 			(show_name no)
@@
 		)
 		(property "Description" "Power symbol creates a global label with name \"+48V\""
-			(at 251.46 30.48 0)
+			(at 292.1 31.75 0)
 			(hide yes)
 			(show_name no)
@@
 	(symbol
 		(lib_id "power:GND")
+		(at 203.2 41.91 0)
+		(unit 1)
+		(body_style 1)
+		(exclude_from_sim no)
+		(in_bom yes)
+		(on_board yes)
+		(in_pos_files yes)
+		(dnp no)
+		(fields_autoplaced yes)
+		(property "Reference" "#PWR057"
+			(at 203.2 48.26 0)
+			(hide yes)
+			(show_name no)
+			(do_not_autoplace no)
+			(effects
+				(font
+					(size 1.27 1.27)
+				)
+			)
+		)
+		(property "Value" "GND_SPEED"
+			(at 203.2 46.99 0)
+			(show_name no)
+			(do_not_autoplace no)
+			(effects
+				(font
+					(size 1.27 1.27)
+				)
+			)
+		)
+		(property "Footprint" ""
+			(at 203.2 41.91 0)
+			(hide yes)
+			(show_name no)
+			(do_not_autoplace no)
+			(effects
+				(font
+					(size 1.27 1.27)
+				)
+			)
+		)
+		(property "Datasheet" ""
+			(at 203.2 41.91 0)
+			(hide yes)
+			(show_name no)
+			(do_not_autoplace no)
+			(effects
+				(font
+					(size 1.27 1.27)
+				)
+			)
+		)
+		(property "Description" "Power symbol creates a global label with name \"GND\" , ground"
+			(at 203.2 41.91 0)
+			(hide yes)
+			(show_name no)
+			(do_not_autoplace no)
+			(effects
+				(font
+					(size 1.27 1.27)
+				)
+			)
+		)
+		(pin "1"
+		)
+		(instances
+			(project "DataManager_Shield"
+				(path "/74a95295-856f-462a-99dc-2eba26429db4/3f3103c2-6ce4-4371-b040-f30e7a818592"
+					(reference "#PWR057")
+					(unit 1)
+				)
+			)
+		)
+	)
+	(symbol
+		(lib_id "power:GND")
 		(at 173.99 86.36 0)
 		(unit 1)
@@
 			)
 		)
-		(property "Value" "GND"
+		(property "Value" "GND_SPEED"
 			(at 92.71 220.98 0)
 			(show_name no)
@@
 	(symbol
 		(lib_id "Connector_Generic:Conn_02x08_Top_Bottom")
-		(at 238.76 38.1 0)
+		(at 279.4 39.37 0)
 		(unit 1)
 		(body_style 1)
@@
 		(fields_autoplaced yes)
 		(property "Reference" "J3"
-			(at 240.03 24.13 0)
+			(at 280.67 25.4 0)
 			(show_name no)
 			(do_not_autoplace no)
@@
 		)
 		(property "Value" "CAR_OUT"
-			(at 240.03 26.67 0)
+			(at 280.67 27.94 0)
 			(show_name no)
 			(do_not_autoplace no)
@@
 		)
 		(property "Footprint" "Connector_Molex:Molex_Mini-Fit_Jr_5569-16A2_2x08_P4.20mm_Horizontal"
-			(at 238.76 38.1 0)
+			(at 279.4 39.37 0)
 			(hide yes)
 			(show_name no)
@@
 		)
 		(property "Datasheet" ""
-			(at 238.76 38.1 0)
+			(at 279.4 39.37 0)
 			(hide yes)
 			(show_name no)
@@
 		)
 		(property "Description" "Generic connector, double row, 02x08, top/bottom pin numbering scheme (row 1: 1...pins_per_row, row2: pins_per_row+1 ... num_pins), script generated (kicad-library-utils/schlib/autogen/connector/)"
-			(at 238.76 38.1 0)
+			(at 279.4 39.37 0)
 			(hide yes)
 			(show_name no)
@@
 		)
 		(property "JLCPCB Part #" "C485577"
-			(at 238.76 38.1 0)
+			(at 279.4 39.37 0)
 			(hide yes)
 			(show_name no)
@@
 		)
 		(property "FT Rotation Offset" "180"
-			(at 238.76 38.1 0)
+			(at 279.4 39.37 0)
 			(hide yes)
 			(show_name no)
@@
 			)
 		)
-		(property "Value" "GND"
-			(at 77.47 232.41 0)
+		(property "Value" "GND_SPEED"
+			(at 80.01 228.5999 0)
 			(show_name no)
 			(do_not_autoplace no)
@@
 					(size 1.27 1.27)
 				)
+				(justify left)
 			)
 		)

Commit message: Data logger board Major Fixes - Remove Speed Sensor's LED and increase R value - Remove Pedal level reader - Remove aux pin header from BoM, self soldering
Parts:
- removed D10: LED, LED_SMD:LED_0603_1608Metric, symbol Device:LED
- removed D3: BAT54S, Package_TO_SOT_SMD:SOT-23, symbol Diode:BAT54S
- removed J6: B-, TerminalBlock_MetzConnect:TerminalBlock_MetzConnect_Type011_RT05502HBLC_1x02_P5.00mm_Horizontal, symbol Connector:Screw_Terminal_01x02
- removed R26: 1.5M, Resistor_SMD:R_0603_1608Metric, symbol Device:R_Small
- removed R27: 1k, Resistor_SMD:R_0603_1608Metric, symbol Device:R_Small
- removed R29: 470, Resistor_SMD:R_1206_3216Metric, symbol Device:R_Small
- removed R5: 1M, Resistor_SMD:R_0603_1608Metric, symbol Device:R_Small
- added R32: 4.7k, Resistor_SMD:R_0603_1608Metric, symbol Device:R_Small
Connections:
- net B- is gone; now on net GND: R19.2, R20.2, R22.2, U1.4, U1.6, U1.8
- net GND: now also U1.2
- net Speed_Sensor: now also R32.1
- net at U1.1: now also R32.2
- net GND_SPEED renamed Speed_Sensor_Return
- net Speed_Sensor_Return: no longer U1.2

Commit message: Isolate B-
Connections:
- net GND: no longer J1.3 (Pin_3), J3.3 (Pin_3), R19.2, R20.2, R22.2, U1.2, U1.4, U1.6, U1.8
- new net B-: J1.3 (Pin_3), J3.3 (Pin_3), R19.2, R20.2, R22.2, U1.2, U1.4, U1.6, U1.8
