File: MotorBrake_PCB/MCU.kicad_sch (KiCad schematic)
At the start: 26 parts, among them IC1 ESDA6V1L, J1 ST-LINK, SW2 SW_Push, SW3 SW_Push, U6 STM32G474RETx, X1 NX2016SA-32MHZ

Commit message: up
Connections:
- net PC13 renamed EMER
Changed lines of the file:
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@@
 	)
 	(junction
+		(at 154.94 121.92)
+		(diameter 0)
+		(color 0 0 0 0)
+	)
+	(junction
 		(at 196.85 55.88)
 		(diameter 0)
@@
 	(wire
 		(pts
-			(xy 177.8 83.82) (xy 181.61 83.82)
-		)
-		(stroke
-			(width 0)
-			(type default)
-		)
-	)
-	(wire
-		(pts
 			(xy 105.41 38.1) (xy 105.41 44.45)
 		)
@@
 	(wire
 		(pts
+			(xy 146.05 121.92) (xy 154.94 121.92)
+		)
+		(stroke
+			(width 0)
+			(type default)
+		)
+	)
+	(wire
+		(pts
 			(xy 152.4 58.42) (xy 165.1 58.42)
 		)
@@
 		)
 	)
-	(hierarchical_label "WDO"
-		(shape input)
-		(at 177.8 83.82 180)
-		(effects
-			(font
-				(size 1.27 1.27)
-			)
-			(justify right)
-		)
-	)
 	(hierarchical_label "ADC1_IN4"
 		(shape input)
@@
 		)
 	)
+	(hierarchical_label "WDO"
+		(shape input)
+		(at 181.61 83.82 180)
+		(effects
+			(font
+				(size 1.27 1.27)
+			)
+			(justify right)
+		)
+	)
 	(hierarchical_label "ADC_CURRENT"
 		(shape input)
@@
 		(effects
 			(font
+				(size 1.27 1.27)
+			)
+			(justify right)
+		)
+	)
+	(hierarchical_label "EMER"
+		(shape input)
+		(at 146.05 121.92 180)
+		(effects
+			(font
