File: MotorBrake_PCB/MotorBrake_PCB.kicad_sch (KiCad schematic)
At the start: 6 parts

Commit message: up
Other:
- sheet MCU ports: added EMER; removed none
- sheet ServoBrake ports: added EMER; removed none
Changed lines of the file:
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@@
+	(wire
+		(pts
+			(xy 160.02 121.92) (xy 181.61 121.92)
+		)
+		(stroke
+			(width 0)
+			(type default)
+		)
+	)
 	(wire
 		(pts
@@
 	(wire
 		(pts
+			(xy 160.02 140.97) (xy 181.61 140.97)
+		)
+		(stroke
+			(width 0)
+			(type default)
+		)
+	)
+	(wire
+		(pts
 			(xy 160.02 134.62) (xy 181.61 134.62)
 		)
@@
 		(pts
 			(xy 107.95 82.55) (xy 128.27 82.55)
-		)
-		(stroke
-			(width 0)
-			(type default)
-		)
-	)
-	(wire
-		(pts
-			(xy 160.02 121.92) (xy 181.61 121.92)
 		)
 		(stroke
@@
 			)
 		)
+		(pin "EMER" input
+			(at 160.02 140.97 0)
+			(effects
+				(font
+					(size 1.27 1.27)
+				)
+				(justify right)
+			)
+		)
 		(instances
 			(project "MotorBrake_PCB"
@@
 			(effects
 				(font
+					(size 1.27 1.27)
+				)
+				(justify left)
+			)
+		)
+		(pin "EMER" output
+			(at 181.61 140.97 180)
+			(effects
+				(font
