File: MotorBrake_PCB/MotorBrake_PCB.kicad_pcb (KiCad board)
At the start: 4 copper layers, 70 x 78 mm, 105 parts, among them CN1 XT30(2+2)PB-M.G.B, CN2 24V IN, CN3 EMER, IC1 ESDA6V1L, J1 ST-LINK, J2 aux_pin, J4 CAN_IN, J5 CAN_OUT, Q1 AO3400A, SW1 SMWE-02R-TP, SW2 SW_Push, SW3 SW_Push, U1 74LVC1G08, U2 INA240A2D, U3 TPS3430WDRC, U4 TPS62932, U5 TCAN332, U6 STM32G474RETx, U7 LM1117MP-3.3, X1 NX2016SA-32MHZ

Commit message: up
Parts:
- removed kibuzzard-6A10704C: G***, kibuzzard-6A10704C
- added R19: 470, Resistor_SMD:R_0603_1608Metric, F.Cu at (97.0, 128.5)
- added R20: 470, Resistor_SMD:R_0603_1608Metric, F.Cu at (97.0, 131.5)
- added R6: 10k, Resistor_SMD:R_0402_1005Metric, F.Cu at (118.0, 90.5)
- added R7: 10k, Resistor_SMD:R_0402_1005Metric, F.Cu at (143.5, 112.0)
- added U8: PC817, Package_DIP:DIP-4_W7.62mm, F.Cu at (99.7, 133.5)
- moved CN3 26.1 mm to (93.0, 130.0), turned to 90 degrees
- moved kibuzzard-6A107033 22.7 mm to (96.7, 123.9)
- moved TP1 3.68 mm to (88.5, 128.1)
- moved kibuzzard-6A10703E 1.36 mm to (85.2, 126.5)
- moved D3 1.30 mm to (95.6, 119.0)
Connections:
- CN3 pad 1: Net-(CN3--) -> GND
- D1 pad 2: Net-(CN3-+) -> Net-(D1-A)
- Q1 pad 3: Net-(CN3--) -> Net-(D1-A)
- RLY1 pad 4: Net-(CN3-+) -> Net-(D1-A)
Routing:
- net /MCU/PC13: track 68.3 -> 140.7 mm, vias 6 -> 7
- net Net-(D1-A): track 0.00 -> 27.3 mm, vias 0 -> 1
- net Net-(CN3-+): track 23.4 -> 6.01 mm
- net /MCU/RELAY: track 28.0 -> 42.3 mm
- net GND: track 101.3 -> 113.6 mm
- net Net-(CN3--): track 11.0 -> 0.00 mm
- net +24V: track 104.7 -> 97.1 mm, vias 1 -> 0
- net Net-(R20-Pad1): track 0.00 -> 3.21 mm
- net /MCU/WDO: track 80.5 -> 81.9 mm, vias 6 -> 5
- net +3V3: track 40.7 -> 42.0 mm, vias 41 -> 42
- net Net-(R19-Pad1): track 0.00 -> 1.35 mm
